Commit message: mapping launch paramaters updated

File: catkin_ws/src/udacity_bot/urdf/udacity_bot.xacro (robot description, xacro)
@@ -1,183 +1,254 @@
 <?xml version='1.0'?>
-<robot name="udacity_bot" xmlns:xacro="http://www.ros.org/wiki/xacro">
-    <xacro:include filename="$(find udacity_bot)/urdf/udacity_bot.gazebo" />
-    <link name="robot_footprint"></link>
-    <joint name="robot_footprint_joint" type="fixed">
-        <origin xyz="0 0 0" rpy="0 0 0"/>
-        <parent link="robot_footprint"/>
-        <child link="chassis"/>
-    </joint>
-    <link name='left_wheel'>
-        <inertial>
-            <mass value="5.0"/>
-            <origin xyz="0.0 0 0" rpy=" 0 1.5707 1.5707"/>
-            <inertia ixx="0.1" ixy="0" ixz="0" iyy="0.1" iyz="0" izz="0.1"/>
-        </inertial>
-        <collision name='collision'>
-            <origin xyz="0.0 0 0" rpy=" 0 1.5707 1.5707"/>
-            <geometry>
-                <cylinder length="0.05" radius="0.1"/>
-            </geometry>
-        </collision>
-        <visual name='wheel_visual'>
-            <origin xyz="0.0 0 0" rpy=" 0 1.5707 1.5707"/>
-            <geometry>
-                <cylinder length="0.05" radius="0.1"/>
-            </geometry>
-			      <material name="black"/>
-        </visual>
-    </link>
-    <joint type="continuous" name="left_wheel_hinge">
-        <origin xyz="0.0 0.25 0" rpy="0 0 0"/>
-        <child link="left_wheel"/>
-        <parent link="chassis"/>
-        <axis xyz="0 1 0" rpy="0 0 0"/>
-        <limit effort="10000" velocity="1000"/>
-        <joint_properties damping="1.0" friction="1.0"/>
-    </joint>
-    <link name='right_wheel'>
-        <inertial>
-            <mass value="5.0"/>
-            <origin xyz="0.0 0 0" rpy=" 0 1.5707 1.5707"/>
-            <inertia ixx="0.1" ixy="0" ixz="0" iyy="0.1" iyz="0" izz="0.1"/>
-        </inertial>
-        <collision name='collision'>
-            <origin xyz="0.0 0 0" rpy=" 0 1.5707 1.5707"/>
-            <geometry>
-                <cylinder length="0.05" radius="0.1"/>
-            </geometry>
-        </collision>
-        <visual name='wheel_visual'>
-            <origin xyz="0.0 0 0" rpy=" 0 1.5707 1.5707"/>
-            <geometry>
-                <cylinder length="0.05" radius="0.1"/>
-            </geometry>
-			      <material name="black"/>
-        </visual>
-    </link>
-    <joint type="continuous" name="right_wheel_hinge">
-        <origin xyz="0 -0.25 0" rpy="0 0 0"/>
-        <child link="right_wheel"/>
-        <parent link="chassis"/>
-        <axis xyz="0 1 0" rpy="0 0 0"/>
-        <limit effort="10000" velocity="1000"/>
-        <joint_properties damping="1.0" friction="1.0"/>
-    </joint>
-    <link name='camera'>
-        <inertial>
-            <mass value="0.1"/>
-            <origin xyz="0.0 0 0" rpy=" 0 0 0"/>
-            <inertia ixx="1e-6" ixy="0" ixz="0" iyy="1e-6" iyz="0" izz="1e-6"/>
-        </inertial>
-        <collision name='collision'>
-            <origin xyz="0.0 0 0" rpy=" 0 0 0"/>
-            <geometry>
-                <box size="0.05 0.05 0.05"/>
-            </geometry>
-        </collision>
-        <visual name='camera_visual'>
-            <origin xyz="0.0 0 0" rpy=" 0 0 0"/>
-            <geometry>
-                <mesh filename="package://udacity_bot/meshes/kinect.dae"/>
-            </geometry>
-        </visual>
-    </link>
-    <joint type="fixed" name="camera_joint">
-        <origin xyz="0.2 0 0" rpy="0 0 0"/>
-        <child link="camera_rgbd_frame"/>
-        <parent link="camera"/>
-    </joint>
-    <link name="camera_rgbd_frame"/>
-    <link name='hokuyo'>
-        <inertial>
-            <mass value="0.1"/>
-            <origin xyz="0.0 0 0" rpy=" 0 0 0"/>
-            <inertia ixx="1e-6" ixy="0" ixz="0" iyy="1e-6" iyz="0" izz="1e-6"/>
-        </inertial>
-        <collision name='collision'>
-            <origin xyz="0.0 0 0" rpy=" 0 0 0"/>
-            <geometry>
-                <box size="0.1 0.1 0.1"/>
-            </geometry>
-        </collision>
-        <visual name='hokuyo_visual'>
-            <origin xyz="0.0 0 0" rpy=" 0 0 0"/>
-            <geometry>
-                <mesh filename="package://udacity_bot/meshes/hokuyo.dae"/>
-            </geometry>
-        </visual>
-    </link>
-    <joint type="fixed" name="hokuyo_joint">
-        <origin xyz="0.175 0.0 0.1" rpy="0 0 0"/>
-        <child link="hokuyo"/>
-        <parent link="chassis"/>
-    </joint>
-    <link name='chassis'>
-        <pose>0 0 0.1 0 0 0</pose>
-        <inertial>
-            <mass value="15.0"/>
-            <origin xyz="0.0 0 0" rpy=" 0 0 0"/>
-            <inertia ixx="0.1" ixy="0" ixz="0" iyy="0.1" iyz="0" izz="0.1"/>
-        </inertial>
-        <collision name='collision'>
-            <origin xyz="0 0 0" rpy=" 0 0 0"/>
-            <geometry>
-                <box size=".4 .4 .1"/>
-            </geometry>
-        </collision>
-        <visual name='chassis_visual'>
-            <origin xyz="0 0 0" rpy=" 0 0 0"/>
-            <geometry>
-                <box size=".4 .4 .1"/>
-            </geometry>
-			      <material name="blue"/>
-        </visual>
-        <collision name='back_caster_collision'>
-            <origin xyz="-0.15 0 -0.05" rpy=" 0 0 0"/>
-            <geometry>
-                <sphere radius="0.0499"/>
-				        <material name="green"/>
-            </geometry>
-            <surface>
-                <friction>
-                    <ode>
-                        <mu>0</mu>
-                        <mu2>0</mu2>
-                        <slip1>1.0</slip1>
-                        <slip2>1.0</slip2>
-                    </ode>
-                </friction>
-            </surface>
-        </collision>
-        <visual name='back_caster_visual'>
-            <origin xyz="-0.15 0 -0.05" rpy=" 0 0 0"/>
-            <geometry>
-                <sphere radius="0.05"/>
-				        <material name="green"/>
-            </geometry>
-        </visual>
-        <collision name='front_caster_collision'>
-            <origin xyz="0.15 0 -0.05" rpy=" 0 0 0"/>
-            <geometry>
-                <sphere radius="0.0499"/>
-            </geometry>
-            <surface>
-                <friction>
-                    <ode>
-                        <mu>0</mu>
-                        <mu2>0</mu2>
-                        <slip1>1.0</slip1>
-                        <slip2>1.0</slip2>
-                    </ode>
-                </friction>
-            </surface>
-        </collision>
-        <visual name='front_caster_visual'>
-            <origin xyz="0.15 0 -0.05" rpy=" 0 0 0"/>
-            <geometry>
-                <sphere radius="0.05"/>
-				        <material name="green"/>
-            </geometry>
-        </visual>
-    </link>
+<robot name="slam_bot" xmlns:xacro="http://www.ros.org/wiki/xacro">
+  <xacro:include filename="$(find slam_project)/urdf/slam_bot.gazebo" />
+  <link name="robot_footprint"></link>
+  <joint name="robot_footprint_joint" type="fixed">
+    <origin xyz="0 0 0" rpy="0 0 0" />
+    <parent link="robot_footprint"/>
+    <child link="chassis" />
+  </joint>
+  <link name='chassis'>
+    <pose>0 0 0.1 0 0 0</pose>
+    <inertial>
+      <mass value="25.0"/>
+      <origin xyz="0.0 0 0" rpy=" 0 0 0"/>
+      <inertia
+          ixx="0.1" ixy="0" ixz="0"
+          iyy="0.1" iyz="0"
+          izz="0.1"
+      />
+    </inertial>
+    <collision name='chassis_collision'>
+      <origin xyz="0 0 0" rpy=" 0 0 0"/>
+      <geometry>
+        <box size=".4 .2 .1"/>
+      </geometry>
+    </collision>
+    <visual name='chassis_visual'>
+      <origin xyz="0 0 0" rpy=" 0 0 0"/>
+      <geometry>
+        <box size=".4 .2 .1"/>
+      </geometry>
+    </visual>
+    <collision name='front_chassis_collision'>
+      <origin xyz="0.2 0 0" rpy=" 0 0 0"/>
+      <geometry>
+        <box size=".3 .08 .04"/>
+      </geometry>
+    </collision>
+    <visual name='front_chassis_visual'>
+      <origin xyz="0.2 0 0" rpy=" 0 0 0"/>
+      <geometry>
+        <box size=".3 .08 .04"/>
+      </geometry>
+    </visual>
+    <collision name='driver_collision'>
+      <origin xyz="0.12 0 0.04" rpy=" 0 1.5707 1.5707"/>
+      <geometry>
+        <cylinder radius=".08" length="0.199"/>
+      </geometry>
+    </collision>
+    <visual name='driver_visual'>
+      <origin xyz="0.12 0 0.04" rpy=" 0 1.5707 1.5707"/>
+      <geometry>
+        <cylinder radius=".08" length="0.199"/>
+      </geometry>
+    </visual>
+    <collision name='connector_collision'>
+      <origin xyz="0.32 0 0" rpy=" 0 1.5707 1.5707"/>
+      <geometry>
+        <cylinder radius=".01" length="0.16"/>
+      </geometry>
+    </collision>
+    <visual name='connector_visual'>
+      <origin xyz="0.32 0 0" rpy=" 0 1.5707 1.5707"/>
+      <geometry>
+        <cylinder radius=".01" length="0.16"/>
+      </geometry>
+    </visual>
+    <collision name='back_caster_collision'>
+      <origin xyz="-0.15 0 -0.05" rpy=" 0 0 0"/>
+      <geometry>
+        <sphere radius="0.0499"/>
+      </geometry>
+    </collision>
+    <visual name='back_caster_visual'>
+      <origin xyz="-0.15 0 -0.05" rpy=" 0 0 0"/>
+      <geometry>
+        <sphere radius="0.05"/>
+      </geometry>
+    </visual>
+    <collision name='front_caster_collision'>
+      <origin xyz="0.15 0 -0.05" rpy=" 0 0 0"/>
+      <geometry>
+        <sphere radius="0.0499"/>
+      </geometry>
+    </collision>
+    <visual name='front_caster_visual'>
+      <origin xyz="0.15 0 -0.05" rpy=" 0 0 0"/>
+      <geometry>
+        <sphere radius="0.05"/>
+      </geometry>
+    </visual>
+    <visual name='back_left_shield_visual'>
+      <origin xyz="-0.15 -0.089 0.08" rpy=" 0 0 0"/>
+      <geometry>
+        <box size=".1 .02 .12"/>
+      </geometry>
+    </visual>
+    <visual name='back_right_shield_visual'>
+      <origin xyz="-0.15 0.089 0.08" rpy=" 0 0 0"/>
+      <geometry>
+        <box size=".1 .02 .12"/>
+      </geometry>
+    </visual>
+    <visual name='back_shield1_visual'>
+      <origin xyz="-0.19 0.0 0.12" rpy=" 0 1.5707 1.5707"/>
+      <geometry>
+        <cylinder radius="0.01"  length="0.18"/>
+      </geometry>
+    </visual>
+    <visual name='back_shield2_visual'>
+      <origin xyz="-0.16 0.0 0.1" rpy=" 0 1.5707 1.5707"/>
+      <geometry>
+        <cylinder radius="0.01"  length="0.18"/>
+      </geometry>
+    </visual>
+    <visual name='back_shield3_visual'>
+      <origin xyz="-0.13 0.0 0.08" rpy=" 0 1.5707 1.5707"/>
+      <geometry>
+        <cylinder radius="0.01"  length="0.18"/>
+      </geometry>
+    </visual>
+  </link>
+  <link name="left_wheel">
+    <inertial>
+      <mass value="5.0"/>
+      <origin xyz="0.0 0 0" rpy=" 0 1.5707 1.5707"/>
+      <inertia
+          ixx="0.1" ixy="0" ixz="0"
+          iyy="0.1" iyz="0"
+          izz="0.1"
+      />
+    </inertial>
+    <collision name='collision'>
+      <origin xyz="0.0 0 0" rpy=" 0 1.5707 1.5707"/>
+      <geometry>
+        <cylinder radius="0.1" length="0.05"/>
+      </geometry>
+    </collision>
+    <visual name='left_wheel_visual'>
+      <origin xyz="0.0 0 0" rpy=" 0 1.5707 1.5707"/>
+      <geometry>
+        <cylinder radius="0.1" length="0.05"/>
+      </geometry>
+    </visual>
+  </link>
+  <joint type="continuous" name="left_wheel_hinge">
+    <origin xyz="0 0.15 0" rpy="0 0 0"/>
+    <child link="left_wheel"/>
+    <parent link="chassis"/>
+    <axis xyz="0 1 0" rpy="0 0 0"/>
+    <limit effort="10000" velocity="1000"/>
+    <dynamics damping="1.0" friction="1.0"/>
+  </joint>
+  <link name="right_wheel">
+    <inertial>
+      <mass value="5.0"/>
+      <origin xyz="0.0 0 0" rpy=" 0 1.5707 1.5707"/>
+      <inertia
+          ixx="0.1" ixy="0" ixz="0"
+          iyy="0.1" iyz="0"
+          izz="0.1"
+      />
+    </inertial>
+    <collision name='collision'>
+      <origin xyz="0.0 0 0" rpy=" 0 1.5707 1.5707"/>
+      <geometry>
+        <cylinder radius="0.1" length="0.05"/>
+      </geometry>
+    </collision>
+    <visual name='right_wheel_visual'>
+      <origin xyz="0.0 0 0" rpy=" 0 1.5707 1.5707"/>
+      <geometry>
+        <cylinder radius="0.1" length="0.05"/>
+      </geometry>
+    </visual>
+  </link>
+  <joint type="continuous" name="right_wheel_hinge">
+    <origin xyz="0 -0.15 0" rpy="0 0 0"/>
+    <child link="right_wheel"/>
+    <parent link="chassis"/>
+    <axis xyz="0 1 0" rpy="0 0 0"/>
+    <limit effort="10000" velocity="1000"/>
+    <dynamics damping="1.0" friction="1.0"/>
+  </joint>
+  <link name="camera">
+    <inertial>
+      <mass value="0.1"/>
+      <origin xyz="0.0 0 0" rpy=" 0 0 0"/>
+      <inertia
+          ixx="1e-6" ixy="0" ixz="0"
+          iyy="1e-6" iyz="0"
+          izz="1e-6"
+      />
+    </inertial>
+    <collision name='collision'>
+      <origin xyz="0.0 0 0" rpy=" 0 0 0"/>
+      <geometry>
+        <box size="0.05 0.05 0.05"/>
+      </geometry>
+    </collision>
+    <visual name='camera_visual'>
+      <origin xyz="0.0 0 0" rpy=" 0 0 0"/>
+      <geometry>
+        <box size="0.05 0.05 0.05"/>
+      </geometry>
+    </visual>
+  </link>
+  <joint type="fixed" name="camera_joint">
+    <origin xyz="0.35 0 0" rpy="0 0 0"/>
+    <child link="camera"/>
+    <parent link="chassis"/>
+    <axis xyz="0 1 0" rpy="0 0 0"/>
+    <limit effort="10000" velocity="1000"/>
+    <dynamics damping="1.0" friction="1.0"/>
+  </joint>
+  <link name="camera_rgbd_frame"></link>
+  <joint name="camera_rgbd_joint" type="fixed">
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
Commit message: mapping launch paramaters updated

File: catkin_ws/src/udacity_bot/urdf/udacity_bot.xacro (robot description, xacro)
@@ -1,4 +1,4 @@
 <?xml version='1.0'?>
-<robot name="slam_bot" xmlns:xacro="http://www.ros.org/wiki/xacro">
+<robot name="udacity_bot" xmlns:xacro="http://www.ros.org/wiki/xacro">
   <xacro:include filename="$(find udacity_bot)/urdf/udacity_bot.gazebo" />
   <link name="robot_footprint"></link>
@@ -240,5 +240,5 @@
       <origin xyz="0.0 0 0" rpy=" 0 0 0"/>
       <geometry>
-        <mesh filename="package://slam_project/meshes/hokuyo.dae"/>
+        <mesh filename="package://udacity_bot/meshes/hokuyo.dae"/>
       </geometry>
     </visual>

Commit message: start shell script added

File: catkin_ws/src/udacity_bot/urdf/udacity_bot.xacro (robot description, xacro)
@@ -43,16 +43,4 @@
       </geometry>
     </visual>
-    <collision name='driver_collision'>
-      <origin xyz="0.12 0 0.04" rpy=" 0 1.5707 1.5707"/>
-      <geometry>
-        <cylinder radius=".08" length="0.199"/>
-      </geometry>
-    </collision>
-    <visual name='driver_visual'>
-      <origin xyz="0.12 0 0.04" rpy=" 0 1.5707 1.5707"/>
-      <geometry>
-        <cylinder radius=".08" length="0.199"/>
-      </geometry>
-    </visual>
     <collision name='connector_collision'>
       <origin xyz="0.32 0 0" rpy=" 0 1.5707 1.5707"/>
@@ -89,34 +77,4 @@
       <geometry>
         <sphere radius="0.05"/>
-      </geometry>
-    </visual>
-    <visual name='back_left_shield_visual'>
-      <origin xyz="-0.15 -0.089 0.08" rpy=" 0 0 0"/>
-      <geometry>
-        <box size=".1 .02 .12"/>
-      </geometry>
-    </visual>
-    <visual name='back_right_shield_visual'>
-      <origin xyz="-0.15 0.089 0.08" rpy=" 0 0 0"/>
-      <geometry>
-        <box size=".1 .02 .12"/>
-      </geometry>
-    </visual>
-    <visual name='back_shield1_visual'>
-      <origin xyz="-0.19 0.0 0.12" rpy=" 0 1.5707 1.5707"/>
-      <geometry>
-        <cylinder radius="0.01"  length="0.18"/>
-      </geometry>
-    </visual>
-    <visual name='back_shield2_visual'>
-      <origin xyz="-0.16 0.0 0.1" rpy=" 0 1.5707 1.5707"/>
-      <geometry>
-        <cylinder radius="0.01"  length="0.18"/>
-      </geometry>
-    </visual>
-    <visual name='back_shield3_visual'>
-      <origin xyz="-0.13 0.0 0.08" rpy=" 0 1.5707 1.5707"/>
-      <geometry>
-        <cylinder radius="0.01"  length="0.18"/>
       </geometry>
     </visual>
@@ -203,5 +161,5 @@
       <origin xyz="0.0 0 0" rpy=" 0 0 0"/>
       <geometry>
-        <box size="0.05 0.05 0.05"/>
+        <mesh filename="package://udacity_bot/meshes/kinect.dae"/>
       </geometry>
     </visual>
